File: CubeProFanLedCtrlBoard/CubeProFanLedCtrlBoard.sch (KiCad schematic (older format))
At the start: 23 parts, among them J1 Conn_01x02, J10 Conn_01x01, J11 Conn_01x02, J12 Conn_01x02, J13 Conn_01x04, J14 Conn_01x04, J15 Conn_01x04, J16 Conn_02x04_Top_Bottom, J2 Screw_Terminal_01x02, J3 Conn_01x02, J4 Conn_01x03, J5 Conn_01x02, J6 Conn_01x02, J7 Conn_01x01, J8 Conn_01x01, J9 Conn_01x01, Q1 IRF540N, Q2 IRF540N, Q3 IRF540N, Q4 IRF540N, U1 L7812, U2 L7805, U3 L7812

Commit message: Moved A3 and A4 to correct pin
Parts:
- J1: renamed from J2; footprint TerminalBlock_RND:TerminalBlock_RND_205-00045_1x02_P5.00mm_Horizontal -> TerminalBlock_RND:TerminalBlock_RND_205-00067_1x02_P7.50mm_Horizontal
- J10: renamed from J16; value Conn_02x04_Top_Bottom -> Conn_02x04_Odd_Even; symbol Connector_Generic:Conn_02x04_Top_Bottom -> Connector_Generic:Conn_02x04_Odd_Even
- J4: footprint Connector_PinSocket_2.54mm:PinSocket_1x03_P2.54mm_Horizontal -> Connector_PinSocket_2.54mm:PinSocket_1x03_P2.54mm_Vertical
- Q1, Q2, Q3, Q4: value IRF540N -> BUZ11
- U1, U3: value L7812 -> L7805
- renumbered J7 to J11, J8 to J12, J9 to J13, J10 to J14, J11 to J15, J12 to J16, J1 to J2, J13 to J5, J14 to J6, J15 to J7, J5 to J8, J6 to J9
